Commit message: add some small improvements for gazebo simulation

File: urdf/pioneer3dx.xacro (robot description, xacro)
@@ -30,5 +30,5 @@
 		</collision>
 		<inertial>
-		  <mass value="5.67"/>
+		  <mass value="20.00"/>
 		  <inertia ixx="0.07" ixy="0" ixz="0"
 		    iyy="0.08" iyz="0"

Commit message: improve urdf model

File: urdf/pioneer3dx.xacro (robot description, xacro)
@@ -23,16 +23,14 @@
     </visual>
     <collision>
-			<origin xyz="0 0 0" rpy="0 0 0"/>
-			<geometry>
-				<mesh filename="package://pioneer_description/meshes/p3dx_meshes/chassis.stl"/>
-				<!--box size="0.43 0.277 0.17"/-->
-			</geometry>
-		</collision>
-		<inertial>
-		  <mass value="20.00"/>
-		  <inertia ixx="0.07" ixy="0" ixz="0"
-		    iyy="0.08" iyz="0"
-		    izz="0.10"
-		  />
+			<origin xyz="0 0 -0.003" rpy="0 0 0"/>
+			<geometry>
+				<!--<mesh filename="package://pioneer_description/meshes/p3dx_meshes/chassis.stl"/>-->
+				<box size="0.35 0.25 0.14" />
+			</geometry>
+		</collision>
+		<inertial>
+      <origin xyz="-0.005 0 -0.148" rpy="0 0 0"/>
+		  <mass value="3.5"/>
+		  <inertia ixx="1" ixy="0" ixz="0" iyy="1" iyz="0" izz="1" />
 		</inertial>
   </link>
@@ -48,7 +46,5 @@
 				<mass value="0.01"/>
 				<origin xyz="0 0 0"/>
-				<inertia ixx="1" ixy="0" ixz="0"
-					 iyy="1" iyz="0"
-	 				izz="1"/>
+				<inertia ixx="1" ixy="0" ixz="0" iyy="1" iyz="0" izz="1" />
 			</inertial>
 			<origin xyz="0 0 0" rpy="0 0 0"/>
@@ -61,6 +57,6 @@
 			<origin xyz="0 0 0" rpy="0 0 0"/>
 			<geometry>
-				<mesh filename="package://pioneer_description/meshes/p3dx_meshes/top.stl"/>
-				<!--box size="0.44 0.38 0.005"/-->
+				<!--<mesh filename="package://pioneer_description/meshes/p3dx_meshes/top.stl"/>-->
+				<box size="0.45 0.38 0.01"/>
 			</geometry>
 		</collision>
@@ -70,7 +66,7 @@
 		<origin xyz="-0.185 0 0.055" rpy="0 0 0"/>
 		<axis xyz="0 0 1"/>
-		<!--<anchor xyz="0 0 0"/>
+		<anchor xyz="0 0 0"/>
   	<limit effort="100" velocity="100" k_velocity="0" />
-  	<joint_properties damping="0.0" friction="0.0" />-->
+  	<joint_properties damping="0.0" friction="0.0" />
 		<parent link="base_link"/>
 		<child link="swivel"/>
@@ -80,6 +76,5 @@
 			<mass value="0.1"/>
 			<origin xyz="0 0 0"/>
-			<inertia ixx="0.01" ixy="0" ixz="0"
-				 iyy="0.01" iyz="0" izz="0.01"/>
+			<inertia ixx="0.01" ixy="0" ixz="0" iyy="0.01" iyz="0" izz="0.01" />
   	</inertial>
 	  <visual name="base_visual">
@@ -93,5 +88,6 @@
 		  <origin xyz="0 0 0" rpy="0 0 0"/>
 		  <geometry>
-			  <mesh filename="package://pioneer_description/meshes/p3dx_meshes/swivel.stl"/>
+			  <!--<mesh filename="package://pioneer_description/meshes/p3dx_meshes/swivel.stl"/>-->
+        <box size="0.01 0.01 0.01"/>
 		  </geometry>
 	  </collision>
@@ -115,5 +111,6 @@
 		  <origin xyz="0 0 0" rpy="0 0 0"/>
 		  <geometry>
-			  <mesh filename="package://pioneer_description/meshes/p3dx_meshes/center_hubcap.stl"/>
+			  <!--<mesh filename="package://pioneer_description/meshes/p3dx_meshes/center_hubcap.stl"/>-->
+        <box size="0.01 0.01 0.01"/>
 		  </geometry>
 	  </collision>
@@ -122,7 +119,7 @@
 		<origin xyz="-0.026 0 -0.016" rpy="0 0 0"/>
 		<axis xyz="0 1 0"/>
-		<!--<anchor xyz="0 0 0"/>
-    <limit effort="1000" velocity="1000" k_velocity="0" />
-    <joint_properties damping="0.0" friction="0.0" />-->
+		<anchor xyz="0 0 0"/>
+    <limit effort="100" velocity="100" k_velocity="0" />
+    <joint_properties damping="0.0" friction="0.0" />
 	  <parent link="swivel"/>
 		<child link="center_wheel"/>
@@ -143,8 +140,8 @@
 	  </visual>
 	  <collision>
-		  <origin xyz="0 0 0" rpy="0 0 0"/>
+		  <origin xyz="0 0 0" rpy="${-3.1415927/2} 0 0"/>
 		  <geometry>
-		    <mesh filename="package://pioneer_description/meshes/p3dx_meshes/center_wheel.stl"/>
-			  <!--<cylinder radius="0.0375" length="0.03"/>-->
+		    <!--<mesh filename="package://pioneer_description/meshes/p3dx_meshes/center_wheel.stl"/>-->
+			  <cylinder radius="0.0375" length="0.01"/>
 		  </geometry>
 	  </collision>
@@ -157,9 +154,9 @@
 	<!-- Left Wheel -->
 	<joint name="base_left_wheel_joint" type="continuous">
-		<origin xyz="0 0.155 0.093" rpy="0 0 0"/>
+		<origin xyz="0 0.158 0.091" rpy="0 0 0"/>
 		<axis xyz="0 1 0"/>
-		<!--<anchor xyz="0 0 0"/>
-  	<limit effort="1000" velocity="1000" k_velocity="0" />
-  	<joint_properties damping="0.0" friction="0.0" />-->
+		<anchor xyz="0 0 0"/>
+  	<limit effort="100" velocity="100" />
+  	<joint_properties damping="0.0" friction="0.0" />
 		<parent link="base_link"/>
 		<child link="left_wheel"/>
@@ -167,8 +164,8 @@
 	<link name="left_wheel">
 	  <inertial>
-			<mass value="0.1"/>
-			<origin xyz="0 0 0"/>
-		  <inertia ixx="0.012411765597" ixy="-0.000711733678" ixz="0.00050272983"
-				 iyy="0.015218160428" iyz="-0.000004273467" izz="0.011763977943"/>
+			<mass value="0.5"/>
+			<origin xyz="0 0 0"/>
+		  <inertia ixx="0.012411765597" ixy="0" ixz="0"
+				 iyy="0.015218160428" iyz="0" izz="0.011763977943"/>
   	</inertial>
 		<visual>
@@ -180,8 +177,8 @@
 		</visual>
 		<collision>
-			<origin xyz="0 0 0" rpy="0 0 0"/>
-			<geometry>
-			  <mesh filename="package://pioneer_description/meshes/p3dx_meshes/left_wheel.stl"/>
-				<!--<cylinder radius="0.092" length="0.04"/>-->
+			<origin xyz="0 0 0" rpy="${-3.1415927/2} 0 0"/>
+			<geometry>
+			  <!--<mesh filename="package://pioneer_description/meshes/p3dx_meshes/left_wheel.stl"/>-->
+				<cylinder radius="0.09" length="0.01"/>
 			</geometry>
 		</collision>
@@ -193,4 +190,10 @@
 	</joint>
 	<link name="left_hub">
+    <inertial>
+      <mass value="0.01"/>
+      <origin xyz="0 0 0"/>
+      <inertia ixx="0.012411765597" ixy="0" ixz="0"
+        iyy="0.015218160428" iyz="0" izz="0.011763977943"/>
+    </inertial>
 		<visual>
 			<origin xyz="0 0 0" rpy="0 0 0"/>
@@ -203,5 +206,6 @@
 			<origin xyz="0 0 0" rpy="0 0 0"/>
 			<geometry>
-				<mesh filename="package://pioneer_description/meshes/p3dx_meshes/left_hubcap.stl"/>
+				<!--<mesh filename="package://pioneer_description/meshes/p3dx_meshes/left_hubcap.stl"/>-->
+        <box size="0.01 0.01 0.01"/>
 			</geometry>
 		</collision>
@@ -209,9 +213,9 @@
 	<!-- Right Wheel -->
 	<joint name="base_right_wheel_joint" type="continuous">
-		<origin xyz="0 -0.155 0.093" rpy="0 0 0"/>
+		<origin xyz="0 -0.158 0.091" rpy="0 0 0"/>
 		<axis xyz="0 1 0"/>
-		<!--<anchor xyz="0 0 0"/>
-  	<limit effort="1000" velocity="1000" k_velocity="0" />
-  	<joint_properties damping="0.0" friction="0.0" />-->
+		<anchor xyz="0 0 0"/>
+  	<limit effort="100" velocity="100" />
+  	<joint_properties damping="0.0" friction="0.0" />
 		<parent link="base_link"/>
 		<child link="right_wheel"/>
@@ -219,8 +223,8 @@
 	<link name="right_wheel">
   	<inertial>
-			<mass value="0.1"/>
-			<origin xyz="0 0 0"/>
-			<inertia ixx="0.012411765597" ixy="-0.000711733678" ixz="0.00050272983"
-				 iyy="0.015218160428" iyz="-0.000004273467" izz="0.011763977943"/>
+			<mass value="0.5"/>
+			<origin xyz="0 0 0"/>
+			<inertia ixx="0.012411765597" ixy="0" ixz="0"
+				 iyy="0.015218160428" iyz="0" izz="0.011763977943"/>
   	</inertial>
 		<visual>
@@ -232,8 +236,8 @@
 		</visual>
 		<collision>
-			<origin xyz="0 0 0" rpy="0 0 0"/>
-			<geometry>
-			  <mesh filename="package://pioneer_description/meshes/p3dx_meshes/right_wheel.stl"/>
-				<!--<cylinder radius="0.092" length="0.04"/>-->
+			<origin xyz="0 0 0" rpy="${-3.1415927/2} 0 0"/>
+			<geometry>
+			  <!--<mesh filename="package://pioneer_description/meshes/p3dx_meshes/right_wheel.stl"/>-->
+				<cylinder radius="0.09" length="0.01"/>
 			</geometry>
 		</collision>
@@ -245,4 +249,10 @@
 	</joint>
 	<link name="right_hub">
+    <inertial>
+      <mass value="0.01"/>
+      <origin xyz="0 0 0"/>
+      <inertia ixx="0.012411765597" ixy="0" ixz="0"
+        iyy="0.015218160428" iyz="0" izz="0.011763977943"/>
+    </inertial>
 		<visual>
 			<origin xyz="0 0 0" rpy="0 0 0"/>
@@ -255,5 +265,6 @@
 			<origin xyz="0 0 0" rpy="0 0 0"/>
 			<geometry>
-				<mesh filename="package://pioneer_description/meshes/p3dx_meshes/right_hubcap.stl"/>
+				<!--<mesh filename="package://pioneer_description/meshes/p3dx_meshes/right_hubcap.stl"/>-->
+        <box size="0.01 0.01 0.01"/>
 			</geometry>
 		</collision>
@@ -398,5 +409,5 @@
     <actuator name="motor1">
       <hardwareInterface>hardware_interface/VelocityJointInterface</hardwareInterface>
-      <mechanicalReduction>1</mechanicalReduction>
+      <mechanicalReduction>${624/35 * 80/19}</mechanicalReduction>
     </actuator>
   </transmission>
@@ -408,5 +419,5 @@
     <actuator name="motor2">
       <hardwareInterface>hardware_interface/VelocityJointInterface</hardwareInterface>
-      <mechanicalReduction>1</mechanicalReduction>
+      <mechanicalReduction>${-624/35 * 80/19}</mechanicalReduction>
     </actuator>
   </transmission>

Commit message: Edit Laser Position , Use Fixed Joint to display in RVIZ

File: urdf/pioneer3dx.xacro (robot description, xacro)
@@ -63,8 +63,10 @@
 	</link>
 <!-- Swivel -->
-	<joint name="base_swivel_joint" type="continuous">
+	<joint name="base_swivel_joint" type="fixed">
 		<origin xyz="-0.185 0 0.055" rpy="0 0 0"/>
 		<axis xyz="0 0 1"/>
 		<anchor xyz="0 0 0"/>
+		<parent link="base_link"/>
+		<child link="swivel"/>
   	<limit effort="100" velocity="100" k_velocity="0" />
   	<joint_properties damping="0.0" friction="0.0" />
@@ -116,8 +118,10 @@
 	  </collision>
 	</link>
-	<joint name="swivel_hubcap_joint" type="continuous">
+	<joint name="swivel_hubcap_joint" type="fixed">
 		<origin xyz="-0.026 0 -0.016" rpy="0 0 0"/>
 		<axis xyz="0 1 0"/>
 		<anchor xyz="0 0 0"/>
+		<parent link="swivel"/>
+		<child link="center_wheel"/>
     <limit effort="100" velocity="100" k_velocity="0" />
     <joint_properties damping="0.0" friction="0.0" />
@@ -153,5 +157,5 @@
 	</joint>
 	<!-- Left Wheel -->
-	<joint name="base_left_wheel_joint" type="continuous">
+	<joint name="base_left_wheel_joint" type="fixed">
 		<origin xyz="0 0.158 0.091" rpy="0 0 0"/>
 		<axis xyz="0 1 0"/>
@@ -212,5 +216,5 @@
 	</link>
 	<!-- Right Wheel -->
-	<joint name="base_right_wheel_joint" type="continuous">
+	<joint name="base_right_wheel_joint" type="fixed">
 		<origin xyz="0 -0.158 0.091" rpy="0 0 0"/>
 		<axis xyz="0 1 0"/>
@@ -325,5 +329,5 @@
   <!-- Hokuyo Laser -->
   <joint name="hokuyo_joint" type="fixed">
-    <origin xyz="0 0 0.085" rpy="0 0 0"/>
+    <origin xyz="0 0 0.030" rpy="0 0 3.14"/>
     <parent link="camera_link"/>
     <child link="laser"/>
@@ -359,5 +363,5 @@
       <origin xyz="0 0 0" rpy="0 0 0"/>
       <geometry>
-	      <box size="0.05 0.07 0.10"/>
+	      <box size="0.05 0.07 0.05"/>
       </geometry>
     </collision>
@@ -365,5 +369,5 @@
       <origin xyz="0 0 0" rpy="0 0 0"/>
       <geometry>
-      	<box size="0.05 0.07 0.10"/>
+      	<box size="0.05 0.07 0.05"/>
       </geometry>
       <material name="CameraGreen"/>

Commit message: Add Sonar Frame to Support RosAria

File: urdf/pioneer3dx.xacro (robot description, xacro)
@@ -372,4 +372,29 @@
       </geometry>
       <material name="CameraGreen"/>
+    </visual>
+    <inertial>
+      <mass value="1e-5" />
+      <origin xyz="0 0 0" rpy="0 0 0"/>
+      <inertia ixx="1e-6" ixy="0" ixz="0" iyy="1e-6" iyz="0" izz="1e-6" />
+    </inertial>
+  </link>
+  <!-- SONAR ROSARIA -->
+  <joint name="sonar_rosaria" type="fixed">
+    <origin xyz="0.0 0 0.208" rpy="0 0 0"/>
+    <parent link="base_link"/>
+    <child link="sonar"/>
+  </joint>
+  <link name="sonar">
+    <collision>
+      <origin xyz="0 0 0" rpy="0 0 0"/>
+      <geometry>
+	      <box size="0.05 0.07 0.05"/>
+      </geometry>
+    </collision>
+    <visual>
+      <origin xyz="0 0 0" rpy="0 0 0"/>
+      <geometry>
+      	<box size="0.001 0.001 0.001"/>
+      </geometry>
     </visual>
     <inertial>
